File: hardware/mitsubishi2zigbee.kicad_pcb (KiCad board)
At the start: 2 copper layers, 10 parts, among them J1 Conn_01x05, Q1 BSS138, Q2 BSS138

Commit message: Update KiCad hardware schematic layout and component labels.
Reorganize schematic into functional sections and rename CN105/ESP32-C6 values for clarity.
Parts:
- J1: value Conn_01x05 -> CN105
Changed lines of the file:
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@@
 			)
 		)
-		(property "Value" "Conn_01x05"
+		(property "Value" "CN105"
 			(at 4 4.3 0)
 			(layer "F.Fab")
